File: void_keeb.kicad_pcb (KiCad board)
At the start: 2 copper layers, 56 parts, among them J1 AudioJack3_Ground, U1 ProMicro

Commit message: changes
Parts:
- moved U1 34.0 mm to (151.1, 92.7)
- moved J1 33.6 mm to (160.0, 114.3), turned to 180 degrees
Connections:
- U1 pad 11: Net-(U1-Pad11) -> Net-(D11-Pad1)
- U1 pad 12: Net-(U1-Pad12) -> Net-(D12-Pad1)
- U1 pad 13: Net-(U1-Pad13) -> Net-(D17-Pad1)
- U1 pad 14: Net-(U1-Pad14) -> Net-(D10-Pad1)
- U1 pad 15: Net-(U1-Pad15) -> Net-(D1-Pad1)
- U1 pad 16: Net-(D17-Pad1) -> Net-(U1-Pad16)
- U1 pad 17: Net-(D12-Pad1) -> Net-(U1-Pad17)
- U1 pad 18: Net-(D11-Pad1) -> Net-(U1-Pad18)
- U1 pad 19: Net-(D10-Pad1) -> Net-(U1-Pad19)
- U1 pad 20: Net-(D1-Pad1) -> Net-(J1-PadS)
- U1 pad 21: Net-(J1-PadS) -> Net-(J1-PadR)
- U1 pad 23: Net-(J1-PadR) -> Net-(J1-PadT)
- U1 pad 7: Net-(J1-PadT) -> Net-(U1-Pad7)
- k_1 pad 2: Net-(U1-Pad10) -> Net-(U1-Pad6)
- k_2 pad 2: Net-(U1-Pad11) -> Net-(U1-Pad7)
- k_3 pad 2: Net-(U1-Pad12) -> Net-(U1-Pad8)
- k_4 pad 2: Net-(U1-Pad13) -> Net-(U1-Pad9)
- k_5 pad 2: Net-(U1-Pad14) -> Net-(U1-Pad10)
- k_A1 pad 2: Net-(U1-Pad10) -> Net-(U1-Pad6)
- k_B1 pad 2: Net-(U1-Pad14) -> Net-(U1-Pad10)
- k_C1 pad 2: Net-(U1-Pad12) -> Net-(U1-Pad8)
- k_D1 pad 2: Net-(U1-Pad12) -> Net-(U1-Pad8)
- k_E1 pad 2: Net-(U1-Pad12) -> Net-(U1-Pad8)
- k_F1 pad 2: Net-(U1-Pad13) -> Net-(U1-Pad9)
- k_G1 pad 2: Net-(U1-Pad14) -> Net-(U1-Pad10)
- k_Q1 pad 2: Net-(U1-Pad10) -> Net-(U1-Pad6)
- k_R1 pad 2: Net-(U1-Pad13) -> Net-(U1-Pad9)
- k_S1 pad 2: Net-(U1-Pad11) -> Net-(U1-Pad7)
- k_T1 pad 2: Net-(U1-Pad14) -> Net-(U1-Pad10)
- k_V1 pad 2: Net-(U1-Pad13) -> Net-(U1-Pad9)
- k_W1 pad 2: Net-(U1-Pad11) -> Net-(U1-Pad7)
- k_X1 pad 2: Net-(U1-Pad11) -> Net-(U1-Pad7)
- k_Z1 pad 2: Net-(U1-Pad10) -> Net-(U1-Pad6)
- k_func_1 pad 2: Net-(U1-Pad9) -> Net-(U1-Pad5)
- k_func_2 pad 2: Net-(U1-Pad9) -> Net-(U1-Pad5)
- k_func_3 pad 2: Net-(U1-Pad9) -> Net-(U1-Pad5)
- k_func_4 pad 2: Net-(U1-Pad9) -> Net-(U1-Pad5)
- k_func_5 pad 2: Net-(U1-Pad12) -> Net-(U1-Pad8)
- k_func_6 pad 2: Net-(U1-Pad13) -> Net-(U1-Pad9)
- k_func_7 pad 2: Net-(U1-Pad14) -> Net-(U1-Pad10)
Routing:
- net Net-(U1-Pad5): track 0.00 -> 185.1 mm
- net Net-(D1-Pad1): track 0.00 -> 163.6 mm
- net Net-(U1-Pad6): track 0.00 -> 159.9 mm
- net Net-(U1-Pad8): track 0.00 -> 152.2 mm
- net Net-(D10-Pad1): track 0.00 -> 146.6 mm
- net Net-(U1-Pad7): track 0.00 -> 143.1 mm
- net Net-(U1-Pad9): track 0.00 -> 132.7 mm
- net Net-(U1-Pad10): track 0.00 -> 118.1 mm
- net Net-(D11-Pad1): track 0.00 -> 117.8 mm
- net Net-(D12-Pad1): track 0.00 -> 111.0 mm
- net Net-(D17-Pad1): track 0.00 -> 91.2 mm
- net Net-(J1-PadT): track 0.00 -> 40.1 mm
- net Net-(J1-PadR): track 0.00 -> 32.6 mm
- net Net-(J1-PadS): track 0.00 -> 31.2 mm
- net Net-(D22-Pad2): track 0.00 -> 7.66 mm
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Other:
- board outline added: 135.9 x 115.6 mm

Commit message: changes
Parts:
- added D28: 1N4148, Diodes_THT:D_DO-35_SOD27_P7.62mm_Horizontal, F.Cu at (295.9, 57.3)
- added D29: 1N4148, Diodes_THT:D_DO-35_SOD27_P7.62mm_Horizontal, F.Cu at (295.9, 76.4)
- added D30: 1N4148, Diodes_THT:D_DO-35_SOD27_P7.62mm_Horizontal, F.Cu at (295.9, 95.4)
- added D31: 1N4148, Diodes_THT:D_DO-35_SOD27_P7.62mm_Horizontal, F.Cu at (295.9, 114.5)
- added D32: 1N4148, Diodes_THT:D_DO-35_SOD27_P7.62mm_Horizontal, F.Cu at (276.9, 54.3)
- added D33: 1N4148, Diodes_THT:D_DO-35_SOD27_P7.62mm_Horizontal, F.Cu at (276.9, 73.4)
- added D34: 1N4148, Diodes_THT:D_DO-35_SOD27_P7.62mm_Horizontal, F.Cu at (276.9, 92.4)
- added D35: 1N4148, Diodes_THT:D_DO-35_SOD27_P7.62mm_Horizontal, F.Cu at (276.9, 111.5)
- added D36: 1N4148, Diodes_THT:D_DO-35_SOD27_P7.62mm_Horizontal, F.Cu at (257.8, 51.3)
- added D37: 1N4148, Diodes_THT:D_DO-35_SOD27_P7.62mm_Horizontal, F.Cu at (257.8, 70.4)
- added D38: 1N4148, Diodes_THT:D_DO-35_SOD27_P7.62mm_Horizontal, F.Cu at (257.8, 89.4)
- added D39: 1N4148, Diodes_THT:D_DO-35_SOD27_P7.62mm_Horizontal, F.Cu at (257.8, 108.5)
- added D40: 1N4148, Diodes_THT:D_DO-35_SOD27_P7.62mm_Horizontal, F.Cu at (238.8, 48.3)
- added D41: 1N4148, Diodes_THT:D_DO-35_SOD27_P7.62mm_Horizontal, F.Cu at (238.8, 67.4)
- added D42: 1N4148, Diodes_THT:D_DO-35_SOD27_P7.62mm_Horizontal, F.Cu at (238.8, 86.4)
- added D43: 1N4148, Diodes_THT:D_DO-35_SOD27_P7.62mm_Horizontal, F.Cu at (238.8, 105.5)
- added D44: 1N4148, Diodes_THT:D_DO-35_SOD27_P7.62mm_Horizontal, F.Cu at (219.7, 127.5)
- added D45: 1N4148, Diodes_THT:D_DO-35_SOD27_P7.62mm_Horizontal, F.Cu at (219.7, 51.3)
- added D46: 1N4148, Diodes_THT:D_DO-35_SOD27_P7.62mm_Horizontal, F.Cu at (219.7, 70.4)
- added D47: 1N4148, Diodes_THT:D_DO-35_SOD27_P7.62mm_Horizontal, F.Cu at (219.7, 89.4)
- added D48: 1N4148, Diodes_THT:D_DO-35_SOD27_P7.62mm_Horizontal, F.Cu at (219.7, 108.5)
- added D49: 1N4148, Diodes_THT:D_DO-35_SOD27_P7.62mm_Horizontal, F.Cu at (199.4, 130.5)
- added D50: 1N4148, Diodes_THT:D_DO-35_SOD27_P7.62mm_Horizontal, F.Cu at (200.7, 54.3)
- added D51: 1N4148, Diodes_THT:D_DO-35_SOD27_P7.62mm_Horizontal, F.Cu at (200.7, 73.4)
- added D52: 1N4148, Diodes_THT:D_DO-35_SOD27_P7.62mm_Horizontal, F.Cu at (200.7, 92.4)
- added D53: 1N4148, Diodes_THT:D_DO-35_SOD27_P7.62mm_Horizontal, F.Cu at (200.7, 111.5)
- added D54: 1N4148, Diodes_THT:D_DO-35_SOD27_P7.62mm_Horizontal, F.Cu at (179.1, 138.2)
- added J2: AudioJack3_Ground, xess:PJ-313-TH_mod, F.Cu at (161.3, 114.3)
- added U2: ProMicro, promicro:ProMicro, F.Cu at (170.2, 92.7)
- added k_0: SW_Push, Button_Switch_Keyboard:SW_Cherry_MX1A_1.00u_Plate, F.Cu at (270.5, 46.7)
- added k_6: SW_Push, Button_Switch_Keyboard:SW_Cherry_MX1A_1.00u_Plate, F.Cu at (194.3, 46.7)
- added k_7: SW_Push, Button_Switch_Keyboard:SW_Cherry_MX1A_1.00u_Plate, F.Cu at (213.4, 43.7)
- added k_8: SW_Push, Button_Switch_Keyboard:SW_Cherry_MX1A_1.00u_Plate, F.Cu at (232.4, 40.7)
- added k_9: SW_Push, Button_Switch_Keyboard:SW_Cherry_MX1A_1.00u_Plate, F.Cu at (251.5, 43.7)
- added k_H1: SW_Push, Button_Switch_Keyboard:SW_Cherry_MX1A_1.00u_Plate, F.Cu at (194.3, 84.8)
- added k_I1: SW_Push, Button_Switch_Keyboard:SW_Cherry_MX1A_1.00u_Plate, F.Cu at (232.4, 59.8)
- added k_J1: SW_Push, Button_Switch_Keyboard:SW_Cherry_MX1A_1.00u_Plate, F.Cu at (213.4, 81.8)
- added k_K1: SW_Push, Button_Switch_Keyboard:SW_Cherry_MX1A_1.00u_Plate, F.Cu at (232.4, 78.8)
- added k_L1: SW_Push, Button_Switch_Keyboard:SW_Cherry_MX1A_1.00u_Plate, F.Cu at (251.5, 81.8)
- added k_M1: SW_Push, Button_Switch_Keyboard:SW_Cherry_MX1A_1.00u_Plate, F.Cu at (213.4, 100.9)
- added k_N1: SW_Push, Button_Switch_Keyboard:SW_Cherry_MX1A_1.00u_Plate, F.Cu at (194.3, 103.9)
- added k_O1: SW_Push, Button_Switch_Keyboard:SW_Cherry_MX1A_1.00u_Plate, F.Cu at (251.5, 62.8)
- added k_P1: SW_Push, Button_Switch_Keyboard:SW_Cherry_MX1A_1.00u_Plate, F.Cu at (270.5, 65.8)
- added k_U1: SW_Push, Button_Switch_Keyboard:SW_Cherry_MX1A_1.00u_Plate, F.Cu at (213.4, 62.8)
- added k_Y1: SW_Push, Button_Switch_Keyboard:SW_Cherry_MX1A_1.00u_Plate, F.Cu at (194.3, 65.8)
- added k_func_10: SW_Push, Button_Switch_Keyboard:SW_Cherry_MX1A_1.00u_Plate, F.Cu at (289.6, 87.8)
- added k_func_11: SW_Push, Button_Switch_Keyboard:SW_Cherry_MX1A_1.00u_Plate, F.Cu at (289.6, 106.9)
- added k_func_12: SW_Push, Button_Switch_Keyboard:SW_Cherry_MX1A_1.00u_Plate, F.Cu at (213.4, 119.9)
- added k_func_13: SW_Push, Button_Switch_Keyboard:SW_Cherry_MX1A_1.00u_Plate, F.Cu at (190.2, 125.3)
- added k_func_14: SW_Push, Button_Switch_Keyboard:SW_Cherry_MX1A_1.00u_Plate, F.Cu at (169.0, 136.5)
- added k_func_8: SW_Push, Button_Switch_Keyboard:SW_Cherry_MX1A_1.00u_Plate, F.Cu at (289.6, 49.7)
- added k_func_9: SW_Push, Button_Switch_Keyboard:SW_Cherry_MX1A_1.00u_Plate, F.Cu at (289.6, 68.8)
- added k_sign_1: SW_Push, Button_Switch_Keyboard:SW_Cherry_MX1A_1.00u_Plate, F.Cu at (270.5, 84.8)
- added k_sign_2: SW_Push, Button_Switch_Keyboard:SW_Cherry_MX1A_1.00u_Plate, F.Cu at (270.5, 103.9)
- added k_sign_3: SW_Push, Button_Switch_Keyboard:SW_Cherry_MX1A_1.00u_Plate, F.Cu at (251.5, 100.9)
- added k_sign_4: SW_Push, Button_Switch_Keyboard:SW_Cherry_MX1A_1.00u_Plate, F.Cu at (232.4, 97.9)
- moved D10 11.4 mm to (69.8, 70.3)
- moved D11 11.4 mm to (69.8, 89.4)
- moved D12 11.4 mm to (69.8, 108.4)
- moved D23 11.4 mm to (127.0, 54.3)
- moved D24 11.4 mm to (127.0, 73.3)
- moved D25 11.4 mm to (127.0, 92.4)
- moved D26 11.4 mm to (127.0, 111.4)
- moved D27 11.4 mm to (144.8, 149.9)
- moved D9 11.4 mm to (69.8, 51.3)
- moved J1 11.4 mm to (148.6, 114.3)
- moved U1 11.4 mm to (139.7, 92.7)
- moved k_2 11.4 mm to (63.5, 43.6)
- moved k_3 11.4 mm to (82.5, 40.6)
- moved k_4 11.4 mm to (101.6, 43.6)
- moved k_5 11.4 mm to (120.7, 46.6)
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Routing:
- net Net-(D28-Pad1): track 0.00 -> 159.6 mm
- net Net-(D29-Pad1): track 0.00 -> 149.4 mm
- net Net-(D31-Pad1): track 0.00 -> 147.4 mm
- net Net-(D30-Pad1): track 0.00 -> 103.3 mm
- net Net-(U2-Pad11): track 0.00 -> 102.5 mm
- net Net-(U2-Pad12): track 0.00 -> 96.4 mm
- net Net-(D44-Pad1): track 0.00 -> 91.6 mm
- net Net-(U2-Pad19): track 0.00 -> 89.6 mm
- net Net-(U2-Pad18): track 0.00 -> 57.1 mm
- net Net-(U2-Pad17): track 0.00 -> 57.1 mm
- net Net-(U2-Pad16): track 0.00 -> 57.1 mm
- net Net-(J2-PadT): track 0.00 -> 53.1 mm
- net Net-(J2-PadR): track 0.00 -> 36.8 mm
- net Net-(J2-PadS): track 0.00 -> 35.4 mm
- net Net-(D49-Pad2): track 0.00 -> 7.39 mm
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Other:
- outline, holes or cut-outs redrawn
