File: void_keeb.sch (KiCad schematic (older format))
At the start: 56 parts, among them J1 AudioJack3_Ground, U1 ProMicro

Commit message: changes
Connections:
- wire segments 119 -> 116
Changed lines of the file:
@@
 EESchema Schematic File Version 4
+LIBS:void_keeb-cache
 EELAYER 26 0
 EELAYER END
@@
 Connection ~ 3700 3800
 Wire Wire Line
-	4350 3800 5000 3800
+	4350 3800 4850 3800
 Connection ~ 4350 3800
 Wire Wire Line
@@
 	4350 3000 5000 3000
 Connection ~ 4350 3000
-Wire Wire Line
-	2150 2600 2150 3400
 Connection ~ 2150 3400
 Wire Wire Line
@@
 Connection ~ 2150 4200
 Wire Wire Line
-	2800 2600 2800 3400
+	2800 2600 2800 3250
 Connection ~ 2800 3400
 Wire Wire Line
@@
 	3450 2600 3450 3400
 Connection ~ 3450 3400
-Wire Wire Line
-	3450 4200 3450 4700
 Connection ~ 3450 4200
-Wire Wire Line
-	4100 5000 4100 4850
 Connection ~ 4100 4200
 Wire Wire Line
@@
 	4100 5000 4100 5800
 Connection ~ 4100 5000
-Wire Wire Line
-	4750 5000 4750 5600
 Connection ~ 4750 5000
 Wire Wire Line
@@
 Connection ~ 5400 3400
 Wire Wire Line
-	5400 4200 5400 5000
+	5400 4200 5400 4800
 Wire Wire Line
 	5400 5000 5400 5800
@@
 $EndComp
 Wire Wire Line
-	8000 2850 8500 2850
-Wire Wire Line
-	8000 3050 8150 3050
-Wire Wire Line
-	8150 3050 8150 2950
-Wire Wire Line
-	8150 2950 8500 2950
-Wire Wire Line
-	8500 2750 8500 2400
-Wire Wire Line
-	8500 2400 6450 2400
-Connection ~ 5400 5800
-Wire Wire Line
-	4100 3400 4100 4200
-Wire Wire Line
-	3450 3400 3450 4200
-Connection ~ 4750 5600
-Wire Wire Line
-	4750 5600 4750 5800
-Wire Wire Line
-	4750 4200 4750 5000
-Connection ~ 4100 4850
-Wire Wire Line
-	4100 4850 4100 4200
-Connection ~ 3450 4700
-Wire Wire Line
-	3450 4700 3450 5000
-Wire Wire Line
-	6600 3350 6450 3350
-Wire Wire Line
-	6450 2400 6450 3350
-Wire Wire Line
-	2800 3400 2800 4050
-Wire Wire Line
-	2150 3400 2150 3900
-Wire Wire Line
-	6600 4850 6600 3850
-Wire Wire Line
-	4100 4850 6600 4850
-Wire Wire Line
-	6500 4700 6500 3750
-Wire Wire Line
-	6500 3750 6600 3750
-Wire Wire Line
-	3450 4700 6500 4700
-Wire Wire Line
-	6600 3650 6400 3650
-Wire Wire Line
-	6400 3650 6400 4050
-Wire Wire Line
-	6400 4050 2800 4050
-Connection ~ 2800 4050
-Wire Wire Line
-	2800 4050 2800 4200
-Wire Wire Line
-	6600 3550 6300 3550
-Wire Wire Line
-	6300 3550 6300 3900
-Wire Wire Line
-	6300 3900 2150 3900
-Connection ~ 2150 3900
-Wire Wire Line
-	2150 3900 2150 4200
+	4100 3400 4100 4000
+Wire Wire Line
+	3450 4200 3450 5000
+Wire Wire Line
+	4750 5000 4750 5800
+Wire Wire Line
+	2800 3400 2800 4200
+Wire Wire Line
+	2150 3400 2150 4200
+Connection ~ 2800 2600
+Wire Wire Line
+	2800 2600 2750 2600
+Wire Wire Line
+	4100 4200 4100 5000
+Wire Wire Line
+	4750 4200 4750 4700
+Wire Wire Line
+	3450 3400 3450 3900
+Wire Wire Line
+	6600 3250 2800 3250
+Connection ~ 2800 3250
+Wire Wire Line
+	2800 3250 2800 3400
+Wire Wire Line
+	2150 2600 2150 3150
+Wire Wire Line
+	6600 3150 2150 3150
+Connection ~ 2150 3150
+Wire Wire Line
+	2150 3150 2150 3400
+Wire Wire Line
+	6600 3350 5500 3350
+Wire Wire Line
+	5500 3350 5500 3900
+Wire Wire Line
+	5500 3900 3450 3900
+Connection ~ 3450 3900
+Wire Wire Line
+	3450 3900 3450 4200
+Wire Wire Line
+	6600 3450 5600 3450
+Wire Wire Line
+	5600 3450 5600 4000
+Wire Wire Line
+	5600 4000 4100 4000
+Connection ~ 4100 4000
+Wire Wire Line
+	4100 4000 4100 4200
+Wire Wire Line
+	6600 3550 5700 3550
+Wire Wire Line
+	5700 3550 5700 4700
+Wire Wire Line
+	5700 4700 4750 4700
+Connection ~ 4750 4700
+Wire Wire Line
+	4750 4700 4750 5000
+Wire Wire Line
+	5400 4800 5800 4800
+Wire Wire Line
+	5800 4800 5800 3650
+Wire Wire Line
+	5800 3650 6600 3650
+Connection ~ 5400 4800
+Wire Wire Line
+	5400 4800 5400 5000
+Wire Wire Line
+	5000 5400 6600 5400
+Wire Wire Line
+	6600 5400 6600 3850
+Connection ~ 5000 5400
+Wire Wire Line
+	6600 3750 5900 3750
+Wire Wire Line
+	5900 3750 5900 4600
+Wire Wire Line
+	5900 4600 5000 4600
+Connection ~ 5000 4600
+Wire Wire Line
+	5000 6200 8000 6200
+Wire Wire Line
+	8000 6200 8000 3850
 Connection ~ 5000 6200
 Wire Wire Line
-	8000 3150 8050 3150
-Wire Wire Line
-	8050 3150 8050 4200
-Wire Wire Line
-	8050 4200 5850 4200
-Wire Wire Line
-	5850 4200 5850 3000
-Wire Wire Line
-	5850 3000 5000 3000
+	4850 2100 4850 3800
+Connection ~ 4850 3800
+Wire Wire Line
+	4850 3800 5000 3800
+Wire Wire Line
+	5000 3000 6200 3000
+Wire Wire Line
+	6200 3000 6200 2200
+Wire Wire Line
+	6200 2200 8950 2200
+Wire Wire Line
+	8950 2200 8950 3650
+Wire Wire Line
+	8950 3650 8000 3650
 Connection ~ 5000 3000
 Wire Wire Line
-	5000 3800 5750 3800
-Wire Wire Line
-	5750 3800 5750 4300
-Wire Wire Line
-	5750 4300 8150 4300
-Wire Wire Line
-	8150 4300 8150 3250
-Wire Wire Line
-	8150 3250 8000 3250
-Connection ~ 5000 3800
-Wire Wire Line
-	9300 5800 9300 3750
-Wire Wire Line
-	8000 3750 9300 3750
-Wire Wire Line
-	5400 5800 9300 5800
-Wire Wire Line
-	9200 3850 9200 5600
-Wire Wire Line
-	8000 3850 9200 3850
-Wire Wire Line
-	4750 5600 9200 5600
-Wire Wire Line
-	8000 3350 8250 3350
-Wire Wire Line
-	8250 3350 8250 4600
-Wire Wire Line
-	8250 4600 5000 4600
-Connection ~ 5000 4600
-Wire Wire Line
-	8000 3450 8350 3450
-Wire Wire Line
-	8350 3450 8350 5400
-Wire Wire Line
-	8350 5400 5000 5400
-Connection ~ 5000 5400
-Wire Wire Line
-	8000 3550 8450 3550
-Wire Wire Line
-	8450 3550 8450 6200
-Wire Wire Line
-	8450 6200 5000 6200
+	9050 2100 9050 3750
+Wire Wire Line
+	9050 3750 8000 3750
+Wire Wire Line
+	4850 2100 9050 2100
+Wire Wire Line
+	8500 2750 8250 2750
+Wire Wire Line
+	8250 2750 8250 2850
+Wire Wire Line
+	8250 2850 8000 2850
+Wire Wire Line
+	8500 2850 8300 2850
+Wire Wire Line
+	8300 2850 8300 3050
+Wire Wire Line
+	8300 3050 8000 3050
+Wire Wire Line
+	8000 3150 8500 3150
+Wire Wire Line
+	8500 3150 8500 2950
 $EndSCHEMATC

Commit message: changes
Parts:
- added D28, D29, D30, D31, D32, D33, D34, D35, D36, D37, D38, D39, D40, D41, D42, D43, D44, D45, D46, D47, D48, D49, D50, D51, D52, D53, D54: 1N4148, Diodes_THT:D_DO-35_SOD27_P7.62mm_Horizontal, symbol Diode:1N4148
- added J2: AudioJack3_Ground, xess:PJ-313-TH_mod, symbol Connector:AudioJack3_Ground
- added U2: ProMicro, promicro:ProMicro, symbol promicro:ProMicro
- added k_0, k_6, k_7, k_8, k_9, k_H1, k_I1, k_J1, k_K1, k_L1, k_M1, k_N1, k_O1, k_P1, k_U1, k_Y1, k_func_10, k_func_11, k_func_12, k_func_13, k_func_14, k_func_8, k_func_9, k_sign_1, k_sign_2, k_sign_3, k_sign_4: SW_Push, Button_Switch_Keyboard:SW_Cherry_MX1A_1.00u_Plate, symbol Switch:SW_Push
Connections:
- wire segments 116 -> 232
